File: beacon/SCH/beacon.sch (KiCad schematic (older format))
At the start: 12 parts, among them P1 CONNECTOR, U1 74LS14, U2 LM555N, U3 QFM-TX1

Commit message: PCB modified
Parts:
- removed BT1: BATTERY, Coin Cell Holder:Coin_Cell_Holder_CH25-2032LF, symbol BATTERY
- removed TH1: 1k5, Capacitors_ThroughHole:Capacitor7x3-5RM5_RevB, symbol THERMISTOR
- added J1: HEADER_1x02, Mlab_Pin_Headers:Angled_1x02, symbol HEADER_1x02
- added R3: 1k5, Resistors_SMD:R_0805_HandSoldering, symbol R
- added R? (x2): 0, symbol R
- C1, C2, C3, C4: footprint Capacitors_SMD:C_0805 -> Capacitors_SMD:C_0805_HandSoldering
- P1: footprint Pin_Headers:Pin_Header_Straight_1x01 -> Mlab_Pin_Headers:Angled_1x01
- U1: footprint (none) -> SMD_Packages:SOIC-14_W
Connections:
- wire segments 42 -> 53
Other:
- moved on the sheet: C1, C2, C3, C4, R1, R2
